File: pcb/ledboard.sch (KiCad schematic (older format))
At the start: 68 parts, among them J1 CONN_USB_MINI_B_H_SMD, P1 CONN_2, P2 SMD452 Hombon connector, P3 SMD452 Hombon connector, P4 SMD452 Hombon connector, P5 CONN_3X2, U1 DSPIC33FJ16GS502-I/SO, U5 MCP16301, U6 MCP79410-I/MS, U7 MCP2200_SOIC-20, X1 CRYSTAL, Y1 12MHZ_HC-49-S

Commit message: Diverging into wifi ledboard
Parts:
- removed BT1: BAT-HLD-001 3V COIN CELL, LNX-BAT-HLD-001, symbol BATTERY
- removed C1: 1uF, SM0603, symbol C
- removed C3, C5, C50, C51: 4.7uF, SM0805, symbol C
- removed C33, C48, C49: 18nF, SM0603, symbol C
- removed C38, C39: 18pF, SM0603, symbol C
- removed C4: 4.7uF, SM0603, symbol C
- removed C40, C42: 5pF, SM0603, symbol C
- removed C41: 100pF, SM0603, symbol C
- removed C43: 100nF, SM0603, symbol C
- removed C44, C45, C46, C47: 470pF, SM0603, symbol C
- removed D16, D17, D18, D19: LED, LED-0603, symbol LED
- removed D20: PRTR5V0U2X_SOT-143-B, SOT-143-B, symbol PRTR5V0U2X_SOT-143-B
- removed J1: CONN_USB_MINI_B_H_SMD, CONN_USB_MINI_B_H_SMD, symbol CONN_USB_MINI_B_H_SMD
- removed P2, P3, P4: SMD452 Hombon connector, ~, symbol CONN_SMD
- removed P5: CONN_3X2, TC2030-MCP-NL, symbol CONN_3X2
- removed R1, R32, R33, R34: 10k, SM0603, symbol R
- removed R2, R40: 470, SM0603, symbol R
- removed R24, R35: 0R, SM0603, symbol R
- removed R3: 10k 1%, SM0603, symbol R
- removed R31: 1k, SM0603, symbol R
- removed R4: 2k4 1%, SM0603, symbol R
- removed R41, R42, R43: 1K, SM0603, symbol R
- removed R5: 10R, SM0603, symbol R
- removed U1: DSPIC33FJ16GS502-I/SO, SO28, symbol DSPIC33FJ16GS502-I/SO
- removed U6: MCP79410-I/MS, MSOP-8, symbol MCP7940
- removed U7: MCP2200_SOIC-20, SOIC-20, symbol MCP2200_SOIC-20
- removed X1: CRYSTAL, ABS07-XTAL, symbol CRYSTAL
- removed Y1: 12MHZ_HC-49-S, HC-49-S, symbol 12MHZ_HC-49-S
- removed Z1: NBEE_LOGO, NBEE_LOGO, symbol NBEE_LOGO
- added Z1: MHOLE, MHOLE_3MM, symbol MHOLE
- renumbered C2 to C1, C34 to C2, C35 to C3, C36 to C4, C37 to C5, D15 to D1, D13 to D2, D14 to D3, R39 to R1, R28 to R2, R29 to R3, U5 to U1
Connections:
- net labels removed: /RESET, BUCK1_IREF, BUCK1_VREF, BUCK2_IREF, BUCK2_VREF, BUCK3_IREF, BUCK3_VREF, DGND, IRQ, PGC1, PGD1, PWM1H, PWM1L, PWM2H, PWM2L, PWM3H, PWM3L, SCL, SDA, UART_RX, UART_TX, VBAT, VIN_REF
- wire segments 234 -> 38
- no-connect marks 16 -> 4
Other:
- note removed: "Add: FTDI 3.3V connector for upgrades or MCP2200\n"
- note removed: "External Connector\n"
- note removed: "Fix: RTC Footprint, BAT footprint, PIC footprint, OLED connector invert\n R5->FB\n"
- note removed: "GND join point"
- note removed: "Power DSC"
- note removed: "Power outputs"
- note removed: "Programming\nConnector\n"
- note removed: "RTC Clock and Battery\n"
- note removed: "Reset\nCircuit"
- note removed: "VIN\nreference"
- moved on the sheet: C1, C2, C3, C4, C5, D1, D2, D3, L1, P1, R1, R2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

Commit message: new design, initial version
Parts:
- added C?: 4.7uF, symbol C_Small
- added C? (x3): 100nF, symbol C_Small
- added CON?: BARREL_JACK, symbol BARREL_JACK
- added D?: LED, symbol LED
- added P?: CONN_01X05, symbol CONN_01X05
- added P?: PIR SENSOR, symbol CONN_01X03
- added P? (x4): CONN_2, bornier2, symbol CONN_2
- added P?: CONN_01X03, symbol CONN_01X03
- added Q? (x3): IRF540N, TO-220, symbol IRF540N
- added R?: 470, SM0603, symbol R
- added R? (x6): 10K, SM0603, symbol R
- added R? (x4): 100, SM0603, symbol R
- added R? (x3): 160, SM0603, symbol R
- added SW?: SW_PUSH, symbol SW_PUSH
- added U2: ESP-12E, symbol ESP-12E
Connections:
- net labels added: CHIP_ENABLE, FLASH, GND, PIR_MOTION, PWM_DIMMER1, PWM_DIMMER2, PWM_DIMMER3, RXD, TXD, VIN, VIN_DIV, WAKEUP_RST, WS2812B_DO, _FLASH, _GPIO2, _RXD, _TXD, nLED, nPUSHBUTTON, nRESET
- wire segments 38 -> 112
Other:
- note added: "5V to 15V input"
- note added: "ADDRESSABLE LED STRIP\n5V INPUT ONLY"
- note added: "MOUNTING\nHOLES"
- note added: "PIR SENSOR"
- note added: "PUSH BUTTON"
- note added: "WIFI/MICROPROCESSOR"
- moved on the sheet: P1, Z1, Z2, Z3, Z4
